Commit message: feat(model): 接入银灰软指与 D405 腕部相机
统一 URDF、SRDF 和 MuJoCo 装配，保留源 CAD 与可复现导入工具，更新碰撞、仿真载荷、回归测试和文档。清理一次性检查与渲染程序及临时 CAD 环境。验证：完整回归 1250 passed / 2 skipped、分层 26 passed；提交快照补齐外部测试依赖后相关 21 项复测通过。

File: src/rebotarm_moveit_config/config/rebotarm.urdf (robot description, URDF)
Before this commit: robot reBot-DevArm_fixend, 10 links, 9 joints
Links:
- added link d405_link; collision mesh filename=package://rebotarm_moveit_config/meshes/d405.stl; visual mesh filename=package://rebotarm_moveit_config/meshes/d405.stl
- added link d405_mount_link; collision mesh filename=package://rebotarm_moveit_config/meshes/d405_mount.stl; visual mesh filename=package://rebotarm_moveit_config/meshes/d405_mount.stl
- link left_finger_link: geometry collision mesh filename=package://rebotarm_moveit_config/meshes/left_finger.stl; collision mesh filename=package://rebotarm_moveit_config/meshes/left_soft_gripper_f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
- link right_finger_link: geometry collision mesh filename=package://rebotarm_moveit_config/meshes/right_finger.stl; collision mesh filename=package://rebotarm_moveit_config/meshes/right_soft_gripper_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
Joints:
- added joint d405_joint: type fixed, parent d405_mount_link, child d405_link, origin xyz=0.0010014555241297094 0.06301963080951393 0.011604510071599904 rpy=0.26179625230552039 0 0
- added joint d405_mount_joint: type fixed, parent end_link, child d405_mount_link, origin xyz=-0.08630933 0.0002079068932795 0.0000007587263523 rpy=1.5707963267948966 0 1.5707963267948966
